File: hardware/kicad/espond32-offboard-ssr/espond32-offboard-ssr.kicad_pcb (KiCad board)
At the start: 2 copper layers, 81.5 x 78.9 mm, 68 parts, among them J1 Conn_02x05_Odd_Even, J2 USB_C_Receptacle_USB2.0_16P, J3 Conn_01x02, J4 Conn_01x02, J5 Conn_01x02, J6 Conn_01x02, J7 Conn_01x02, U1 ESP32-S3-WROOM-1-N8, U2 XL1509-3.3

Commit message: Final tweaks before DevKitC deployment
Parts:
- moved J7 3.08 mm to (197.0, 137.0), turned to 90 degrees
- moved J3 3.04 mm to (125.0, 95.0), turned to -90 degrees
- moved J4 3.04 mm to (125.0, 102.0), turned to -90 degrees
- moved J5 3.00 mm to (125.0, 109.0), turned to -90 degrees
- moved J6 3.00 mm to (125.0, 116.0), turned to -90 degrees
Routing:
- net GND: track 480.4 -> 487.9 mm, vias 12 -> 14
- net Net-(D6-COM): track 44.3 -> 46.1 mm
- net Net-(D4-COM): track 27.9 -> 29.2 mm
- net Net-(D5-COM): track 31.8 -> 33.1 mm
- net Net-(D8-COM): track 26.8 -> 27.6 mm

Commit message: updated hardware
Parts:
- L1: footprint Inductor_SMD:L_6.3x6.3_H3 -> Inductor_SMD:L_Sunlord_SWPA6045S
