File: hardware/kicad/espond32-offboard-ssr/espond32-offboard-ssr.kicad_sch (KiCad schematic)
At the start: 0 parts

Commit message: Off-Board SSR hardware may be done...
Parts:
- added C1, C5, C6, C7: 10uF, Capacitor_SMD:C_0603_1608Metric, symbol Device:C_Small_US
- added C10: 10nF, Capacitor_SMD:C_0603_1608Metric, symbol Device:C_Small_US
- added C11: 1uF, Capacitor_SMD:C_0603_1608Metric, symbol Device:C_Small_US
- added C12, C13, C14, C15, C16, C17, C18, C19, C2, C20, C3, C4: 100nF, Capacitor_SMD:C_0603_1608Metric, symbol Device:C_Small_US
- added C8: 100uF, Capacitor_SMD:CP_Elec_6.3x7.7, symbol Device:C
- added C9: 220uF, Capacitor_SMD:CP_Elec_6.3x7.7, symbol Device:C_Small_US
- added D1, D2, D3: ESD9B5.0ST5G, Diode_SMD:D_SOD-923, symbol Diode:ESD9B5.0ST5G
- added D4, D5, D6, D7, D8: BAT54S, Package_TO_SOT_SMD:SOT-23, symbol Diode:BAT54S
- added D9: SS34, Diode_SMD:D_SMA, symbol Diode:SS34
- added D_FLOAT1, D_LIGHT1, D_PUMP1, D_PUMP2, D_SYS1, D_VALVE1: WS2812B-2020, LED_SMD:LED_WS2812B-2020_PLCC4_2.0x2.0mm, symbol LED:WS2812B-2020
- added H1, H2, H3, H4: MountingHole, MountingHole:MountingHole_3.2mm_M3, symbol Mechanical:MountingHole
- added J1: Conn_02x05_Odd_Even, Connector_PinHeader_2.54mm:PinHeader_2x05_P2.54mm_Vertical, symbol Connector_Generic:Conn_02x05_Odd_Even
- added J2: USB_C_Receptacle_USB2.0_16P, Connector_USB:USB_C_Receptacle_HRO_TYPE-C-31-M-12, symbol Connector:USB_C_Receptacle_USB2.0_16P
- added J3, J4, J5, J6, J7: Conn_01x02, TerminalBlock_Phoenix:TerminalBlock_Phoenix_MPT-0,5-2-2.54_1x02_P2.54mm_Horizontal, symbol Connector_Generic:Conn_01x02
- added J_LIGHT1, J_PUMP1, J_PUMP2, J_VALVE1: Conn_01x03, Connector_JST:JST_XH_B3B-XH-A_1x03_P2.50mm_Vertical, symbol Connector_Generic:Conn_01x03
- added L1: 33uH, Inductor_SMD:L_6.3x6.3_H3, symbol Device:L_Small
- added R1, R2: 5.1k, Resistor_SMD:R_0603_1608Metric, symbol Device:R_Small_US
- added R10, R11, R3, R4, R8, R9: 22, Resistor_SMD:R_0603_1608Metric, symbol Device:R_Small_US
- added R12: 330, Resistor_SMD:R_0603_1608Metric, symbol Device:R_Small_US
- added R5: 10k, Resistor_SMD:R_0603_1608Metric, symbol Device:R_Small_US
- added R6: 2.2k, Resistor_SMD:R_0603_1608Metric, symbol Device:R_Small_US
- added R7: 10K, Resistor_SMD:R_0603_1608Metric, symbol Device:R_Small_US
- added SW_GPIO0, SW_MCU_EN1, SW_RESET1: SW_Push, Button_Switch_SMD:SW_SPST_TL3342, symbol Switch:SW_Push
- added U1: ESP32-S3-WROOM-1-N8, RF_Module:ESP32-S3-WROOM-1, symbol RF_Module:ESP32-S3-WROOM-1
- added U2: XL1509-3.3, Package_SO:SOIC-8_3.9x4.9mm_P1.27mm, symbol Regulator_Switching:XL1509-3.3
Connections:
- new net: J2.A5 (CC1), R1.1
- new net: D1.1 (A1), J2.A6 (D+), J2.B6 (D+), R4.1
- new net: D2.1 (A1), J2.A7 (D-), J2.B7 (D-), R3.1
- new net: J2.B5 (CC2), R2.1
- new net: D4.3 (COM), J4.2 (Pin_2), R11.1
- new net: D8.3 (COM), J3.2 (Pin_2), R10.1
- new net: D_PUMP1.3 (DIN), R12.1
- new net: D7.3 (COM), J7.2 (Pin_2), R6.1
- new net: D_LIGHT1.3 (DIN), D_VALVE1.1 (DOUT)
- new net: D_PUMP2.1 (DOUT), D_VALVE1.3 (DIN)
- new net: D5.3 (COM), J5.2 (Pin_2), R9.1
- new net: D_FLOAT1.3 (DIN), D_LIGHT1.1 (DOUT)
- new net: D6.3 (COM), J6.2 (Pin_2), R8.1
- new net: D9.1 (K), L1.1, U2.2 (OUT)
- new net: D_PUMP1.1 (DOUT), D_PUMP2.3 (DIN)
- new net: D_FLOAT1.1 (DOUT), D_SYS1.3 (DIN)
- new net +3V3: C1.2, C14.1, C15.1, C16.1, C17.1, C18.1, C19.1, C2.2, C3.2, C4.2, C7.1, C9.1, D4.2 (K), D5.2 (K), D6.2 (K), D7.2 (K), D8.2 (K), D_FLOAT1.4 (VDD), D_LIGHT1.4 (VDD), D_PUMP1.4 (VDD), D_PUMP2.4 (VDD), D_SYS1.4 (VDD), D_VALVE1.4 (VDD), J_LIGHT1.2 (Pin_2), J_PUMP1.2 (Pin_2), J_PUMP2.2 (Pin_2), J_VALVE1.2 (Pin_2), L1.2, R5.2, R7.2, U1.2 (3V3), U2.3 (FB)
- new net DEBUG_CFG: J1.4 (Pin_4), U1.28 (IO35)
- new net DEBUG_EVAL: J1.5 (Pin_5), U1.39 (IO1)
- new net DEBUG_IO: J1.7 (Pin_7), U1.38 (IO2)
- new net DEBUG_LEAK: J1.10 (Pin_10), U1.31 (IO38)
- new net DEBUG_NET: J1.1 (Pin_1), U1.25 (IO48)
- new net DEBUG_OPERATE: J1.2 (Pin_2), U1.23 (IO21)
- new net DEBUG_RESET: J1.3 (Pin_3), U1.24 (IO47)
- new net DEBUG_SYS_LED: J1.8 (Pin_8), U1.30 (IO37)
- new net DEBUG_TASKS: J1.6 (Pin_6), U1.29 (IO36)
- new net FLOAT_SENS: C10.1, R5.1, R6.2, U1.17 (IO9)
- new net GND: C1.1, C10.2, C11.1, C12.2, C13.2, C14.2, C15.2, C16.2, C17.2, C18.2, C19.2, C2.1, C20.2, C3.1, C4.1, C5.2, C6.2, C7.2, C8.2, C9.2, D1.2 (A2), D2.2 (A2), D3.2 (A2), D4.1 (A), D5.1 (A), D6.1 (A), D7.1 (A), D8.1 (A), D9.2 (A), D_FLOAT1.2 (VSS), D_LIGHT1.2 (VSS), D_PUMP1.2 (VSS), D_PUMP2.2 (VSS), D_SYS1.2 (VSS), D_VALVE1.2 (VSS), J2.A1 (GND), J2.A12 (GND), J2.B1 (GND), J2.B12 (GND), J2.SH (SHIELD), J3.1 (Pin_1), J4.1 (Pin_1), J5.1 (Pin_1), J6.1 (Pin_1), J7.1 (Pin_1), R1.2, R2.2, SW_GPIO0.2, SW_MCU_EN1.2, SW_RESET1.2, U1.1 (GND), U1.40 (GND), U1.41 (GND), U2.4 (~{EN}), U2.5 (GND), U2.6 (GND), U2.7 (GND), U2.8 (GND)
- new net GPIO0: C12.1, SW_GPIO0.1, U1.27 (IO0)
- new net LED_DATA: R12.2, U1.18 (IO10)
- new net LIGHT1_SSR: R8.2, U1.19 (IO11)
- new net LIGHT1_SW_A: J_LIGHT1.3 (Pin_3), U1.20 (IO12)
- new net LIGHT1_SW_B: J_LIGHT1.1 (Pin_1), U1.21 (IO13)
- new net MCU_EN: C11.2, C13.1, R7.1, SW_MCU_EN1.1, U1.3 (EN)
- new net PUMP1_SSR: R10.2, U1.4 (IO4)
- new net PUMP1_SW_A: J_PUMP1.3 (Pin_3), U1.5 (IO5)
- new net PUMP1_SW_B: J_PUMP1.1 (Pin_1), U1.6 (IO6)
- new net PUMP2_SSR: R11.2, U1.7 (IO7)
- new net PUMP2_SW_A: J_PUMP2.3 (Pin_3), U1.8 (IO15)
- new net PUMP2_SW_B: J_PUMP2.1 (Pin_1), U1.9 (IO16)
- new net RESET_BTN: C20.1, SW_RESET1.1, U1.22 (IO14)
- new net USB_D+: R4.2, U1.14 (USB_D+)
- new net USB_D-: R3.2, U1.13 (USB_D-)
- new net VALVE1_SSR: R9.2, U1.10 (IO17)
- new net VALVE1_SW_A: J_VALVE1.3 (Pin_3), U1.11 (IO18)
- new net VALVE1_SW_B: J_VALVE1.1 (Pin_1), U1.12 (IO8)
- new net VBUS: C5.1, C6.1, C8.1, D3.1 (A1), J2.A4 (VBUS), J2.A9 (VBUS), J2.B4 (VBUS), J2.B9 (VBUS), U2.1 (VIN)
- no-connect marks 0 -> 13
Other:
- note added: "Buck Converter 5V -> 3.3V"
- note added: "DEBUG Pin Header"
- note added: "Device Control + LED Indicators"
- note added: "MCU Reset (EN) + Bootloader (GPIO0)"
- note added: "MicroController"
- note added: "Off-Board SSR + Float Sensor Pins"
- note added: "USB-C Interface"

Commit message: updated hardware
Parts:
- L1: footprint Inductor_SMD:L_6.3x6.3_H3 -> Inductor_SMD:L_Sunlord_SWPA6045S
Changed lines of the file:
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@@
 			)
 		)
-		(property "Footprint" "Inductor_SMD:L_6.3x6.3_H3"
+		(property "Footprint" "Inductor_SMD:L_Sunlord_SWPA6045S"
 			(at 158.75 167.64 0)
 			(hide yes)
